File: Test_PCB_design/LED_PCB_Large/LED_PCB_Large.kicad_sch (KiCad schematic)
At the start: 113 parts, among them J1 AS150UPB 2+4, Q1 BUK9Y107-80EX, Q10 BUK9Y107-80EX, Q11 BUK9Y107-80EX, Q12 BUK9Y107-80EX, Q2 BUK9Y107-80EX, Q3 BUK9Y107-80EX, Q4 BUK9Y107-80EX, Q5 BUK9Y107-80EX, Q6 BUK9Y107-80EX, Q7 BUK9Y107-80EX, Q8 BUK9Y107-80EX, Q9 BUK9Y107-80EX, U1 MAX20078ATE_V_T, U2 MAX20078ATE_V_T, U3 MAX20078ATE_V_T, U4 MAX20078ATE_V_T, U5 MAX20078ATE_V_T, U6 MAX20078ATE_V_T

Commit message: updated everything just need to check electrical traces to make sure they work.
Connections:
- removed net LED+: Cout1.1, Cout2.1, Cout3.1, Cout4.1, Cout5.1, Cout6.1, D1.2 (A), D10.2 (A), D12.2 (A), D4.2 (A), D6.2 (A), D8.2 (A), L1.2, L2.2, L3.2, L4.2, L5.2, L6.2, R11.1, R15.1, R19.1, R2.1, R23.1, R7.1
- new net LED1+: Cout6.1, D1.2 (A), L1.2, R2.1
- new net LED2+: Cout1.1, D4.2 (A), L2.2, R7.1
- new net LED3+: Cout2.1, D6.2 (A), L3.2, R11.1
- new net LED4+: Cout3.1, D8.2 (A), L4.2, R15.1
- new net LED5+: Cout4.1, D10.2 (A), L5.2, R19.1
- new net LED6+: Cout5.1, D12.2 (A), L6.2, R23.1
Changed lines of the file:
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@@
 		)
 	)
-	(label "LED+"
+	(label "LED6+"
 		(at 471.17 158.75 0)
 		(effects
@@
 		)
 	)
-	(label "LED+"
+	(label "LED5+"
 		(at 472.44 63.5 0)
 		(effects
@@
 		)
 	)
-	(label "LED+"
+	(label "LED1+"
 		(at 129.54 62.23 0)
 		(effects
@@
 		)
 	)
-	(label "LED+"
+	(label "LED4+"
 		(at 294.64 154.94 0)
 		(effects
@@
 		)
 	)
-	(label "LED+"
+	(label "LED2+"
 		(at 128.27 153.67 0)
 		(effects
@@
 		)
 	)
-	(label "LED+"
+	(label "LED3+"
 		(at 297.18 62.23 0)
 		(effects
