File: LED_PCB_Large/LED_PCB_Large.kicad_pcb (KiCad board)
At the start: 4 copper layers, 85 x 170 mm, 117 parts, among them J1 AS150UPB 2+4, Q1 BUK9Y107-80EX, Q10 BUK9Y107-80EX, Q11 BUK9Y107-80EX, Q12 BUK9Y107-80EX, Q2 BUK9Y107-80EX, Q3 BUK9Y107-80EX, Q4 BUK9Y107-80EX, Q5 BUK9Y107-80EX, Q6 BUK9Y107-80EX, Q7 BUK9Y107-80EX, Q8 BUK9Y107-80EX, Q9 BUK9Y107-80EX, U1 MAX20078ATE_V_T, U2 MAX20078ATE_V_T, U3 MAX20078ATE_V_T, U4 MAX20078ATE_V_T, U5 MAX20078ATE_V_T, U6 MAX20078ATE_V_T

Commit message: Reorganize PCB project and add updated LED PCB design
Parts:
- R11, R15, R19, R2, R23, R7: value 453K 1% -> 324K 1%
- moved R8 0.72 mm to (141.6, 68.9)
Routing:
- net GND: track 163.4 -> 92.0 mm, vias 123 -> 150
- net /PWM: track 359.0 -> 314.3 mm, vias 7 -> 9
- net /LED2+: track 17.3 -> 7.57 mm, vias 2 -> 1
- net /LED3+: track 16.4 -> 7.59 mm, vias 2 -> 1
- net /FAULT: track 386.0 -> 377.6 mm, vias 9 -> 10
- net /LED1+: track 17.0 -> 8.67 mm, vias 2 -> 1
- net /LED6+: track 15.3 -> 7.02 mm, vias 2 -> 1
- net /LED4+: track 16.1 -> 8.35 mm, vias 2 -> 1
- net /LED5+: track 12.9 -> 6.94 mm, vias 2 -> 1
- net Net-(D2-A): track 19.5 -> 17.0 mm
- net Net-(Q10-D_1): track 33.4 -> 31.1 mm
- net Net-(Q1-S_1): track 33.5 -> 31.5 mm
- net Net-(Q9-G): track 5.76 -> 6.71 mm
- net /REF_1V2: track 317.1 -> 317.8 mm
- net +48V_FUSED: track 80.1 -> 80.0 mm, vias 60 -> 68
