File: LED_PCB_Large/LED_PCB_Large.kicad_sch (KiCad schematic)
At the start: 113 parts, among them J1 AS150UPB 2+4, Q1 BUK9Y107-80EX, Q10 BUK9Y107-80EX, Q11 BUK9Y107-80EX, Q12 BUK9Y107-80EX, Q2 BUK9Y107-80EX, Q3 BUK9Y107-80EX, Q4 BUK9Y107-80EX, Q5 BUK9Y107-80EX, Q6 BUK9Y107-80EX, Q7 BUK9Y107-80EX, Q8 BUK9Y107-80EX, Q9 BUK9Y107-80EX, U1 MAX20078ATE_V_T, U2 MAX20078ATE_V_T, U3 MAX20078ATE_V_T, U4 MAX20078ATE_V_T, U5 MAX20078ATE_V_T, U6 MAX20078ATE_V_T

Commit message: Reorganize PCB project and add updated LED PCB design
Parts:
- R11, R15, R19, R2, R23, R7: value 453K 1% -> 324K 1%
Connections:
- no-connect marks 2 -> 0
Changed lines of the file:
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@@
 		(color 0 0 0 0)
 	)
-	(no_connect
-		(at 222.25 234.95)
-	)
-	(no_connect
-		(at 222.25 237.49)
-	)
 	(wire
 		(pts
@@
 			)
 		)
-		(property "Value" "453K 1%"
+		(property "Value" "324K 1%"
 			(at 312.42 63.4999 0)
 			(show_name no)
@@
 			)
 		)
-		(property "Value" "453K 1%"
+		(property "Value" "324K 1%"
 			(at 144.78 63.4999 0)
 			(show_name no)
@@
 			)
 		)
-		(property "Value" "453K 1%"
+		(property "Value" "324K 1%"
 			(at 143.51 154.9399 0)
 			(show_name no)
@@
 		(in_pos_files yes)
 		(dnp no)
-		(fields_autoplaced yes)
 		(property "Reference" "J1"
 			(at 234.95 231.1399 0)
@@
 		)
 		(property "Value" "AS150UPB 2+4"
-			(at 231.14 222.25 0)
+			(at 224.028 218.186 0)
 			(show_name no)
 			(do_not_autoplace no)
@@
 			)
 		)
-		(property "Value" "453K 1%"
+		(property "Value" "324K 1%"
 			(at 487.68 64.7699 0)
 			(show_name no)
@@
 			)
 		)
-		(property "Value" "453K 1%"
+		(property "Value" "324K 1%"
 			(at 309.88 156.2099 0)
 			(show_name no)
@@
 			)
 		)
-		(property "Value" "453K 1%"
+		(property "Value" "324K 1%"
 			(at 486.41 160.0199 0)
 			(show_name no)
